File: hardware/Tiny-RC-Serial.brd (EAGLE design)
At the start: 27.9 x 27.9 mm, 13 parts, among them IC1 ATTINY84A-SSU

Commit message: updated readme and sch and brd
Parts:
- renumbered C3 to C1
Changed lines of the file:
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@@
 <element name="S4" library="SparkFun" package="STAND-OFF-TIGHT" value="STAND-OFFTIGHT" x="3.175" y="24.765"/>
 <element name="S2" library="SparkFun" package="STAND-OFF-TIGHT" value="STAND-OFFTIGHT" x="24.765" y="24.765"/>
-<element name="C3" library="SparkFun" package="CAP-PTH-SMALL" value="0.1uF" x="22.86" y="7.9375" smashed="yes">
+<element name="C1" library="SparkFun" package="CAP-PTH-SMALL" value="0.1uF" x="22.86" y="7.9375" smashed="yes">
 <attribute name="NAME" x="24.13" y="6.35" size="0.6096" layer="25" align="center"/>
 <attribute name="VALUE" x="23.114" y="6.4135" size="0.4064" layer="27"/>
@@
 <signal name="GND">
 <contactref element="JP1" pad="10"/>
-<contactref element="C3" pad="2"/>
+<contactref element="C1" pad="2"/>
 <polygon width="0.254" layer="16">
 <vertex x="1.27" y="26.67"/>
@@
 <signal name="5V">
 <contactref element="JP1" pad="1"/>
-<contactref element="C3" pad="1"/>
+<contactref element="C1" pad="1"/>
 <contactref element="IC1" pad="1"/>
 <wire x1="19.05" y1="5.08" x2="21.59" y2="5.08" width="0.254" layer="16"/>

Commit message: updated to version 3.0
Parts:
- added C2, C3: .22uF, SparkFun-Capacitors:0805
- added Y1: 20Mhz, SparkFun-FreqCtrl:HC49US
- JP3: device jst-ph:JST-PH4 -> SparkFun-Connectors:1X03
- R1: device rcl:R1206 -> SparkFun-Resistors:0805
- moved U$5 25.6 mm to (25.7, 18.1), turned to 90 degrees
- moved LED1 6.63 mm to (3.17, 19.7)
- moved R1 5.24 mm to (6.35, 21.6)
- moved D1 3.86 mm to (7.62, 25.4)
- moved JP3 2.56 mm to (16.5, 25.4)
Connections:
- removed net RST: IC1.4, JP2.5
- removed net RX: IC1.3, JP3.2
- new net N$3: C2.1, IC1.2, Y1.2
- new net N$4: C3.1, IC1.3, Y1.1
- new net RCDATA: IC1.4, JP1.5, JP2.5
- net GND: now also C2.2, C3.2, JP3.1; no longer JP3.4
- net TX: now also IC1.5, JP3.2; no longer IC1.2, JP3.3
- net VIN: now also JP3.3; no longer JP3.1
Routing:
- net RCDATA: track 0.00 -> 31.4 mm, vias 0 -> 3
- net N$4: track 0.00 -> 27.0 mm, vias 0 -> 2
- net N$3: track 0.00 -> 23.3 mm, vias 0 -> 2
- net RST: track 20.9 -> 0.00 mm, vias 2 -> 0
- net GND: track 14.2 -> 30.0 mm, vias 1 -> 2
- net RX: track 9.45 -> 0.00 mm
- net N$1: track 18.4 -> 24.4 mm, vias 1 -> 2
- net N$2: track 3.31 -> 5.65 mm
- net 5V: track 41.8 -> 43.8 mm
- net VIN: track 5.96 -> 4.29 mm
- net RC5: track 26.5 -> 27.9 mm
Other:
- board text added: "(c) 2013 Andy Kipp"
- board text added: "TinyRC Rev 3.0"
- board text removed: "(c) 2012 Andy Kipp"
- board text removed: "6CH RC Serial Interface"
- board text removed: "RX"
- board text removed: "Rev 2.6"
